File: pcb/Nathophone_driver_board.kicad_sch (KiCad schematic)
At the start: 0 parts

Commit message: BEGUN Layout
Other:
- added sheet Data+Power Connections (Nathophone_PCB_Data.kicad_sch)
- added sheet Drivers A (DriversA.kicad_sch)
- added sheet Drivers B (DriversB.kicad_sch)
- added sheet Drivers C (DriversC.kicad_sch)
- added sheet Power (Nathophone_pcb_Power.kicad_sch)
- company: (none) -> Juventus Technikerschule HF
- title: (none) -> Nathophone Driver Board
Changed lines of the file:
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@@
 	(generator_version "9.0")
 	(paper "A4")
+	(title_block
+		(title "Nathophone Driver Board")
+		(date "2025-10-13")
+		(rev "DRAFT")
+		(company "Juventus Technikerschule HF")
+	)
+	(sheet
+		(at 43.18 39.37)
+		(size 27.94 10.16)
+		(exclude_from_sim no)
+		(in_bom yes)
+		(on_board yes)
+		(dnp no)
+		(fields_autoplaced yes)
+		(stroke
+			(width 0.1524)
+			(type solid)
+		)
+		(fill
+			(color 0 0 0 0.0000)
+		)
+		(property "Sheetname" "Power"
+			(at 43.18 38.6584 0)
+			(effects
+				(font
+					(size 1.27 1.27)
+				)
+				(justify left bottom)
+			)
+		)
+		(property "Sheetfile" "Nathophone_pcb_Power.kicad_sch"
+			(at 43.18 50.1146 0)
+			(effects
+				(font
+					(size 1.27 1.27)
+				)
+				(justify left top)
+			)
+		)
+		(instances
+			(project "Nathophone_driver_board"
+				(path "/a109ba74-2574-4a03-88a2-446214ab2b70"
+					(page "2")
+				)
+			)
+		)
+	)
+	(sheet
+		(at 224.155 38.735)
+		(size 40.64 9.525)
+		(exclude_from_sim no)
+		(in_bom yes)
+		(on_board yes)
+		(dnp no)
+		(fields_autoplaced yes)
+		(stroke
+			(width 0.1524)
+			(type solid)
+		)
+		(fill
+			(color 0 0 0 0.0000)
+		)
+		(property "Sheetname" "Drivers C"
+			(at 224.155 38.0234 0)
+			(effects
+				(font
+					(size 1.27 1.27)
+				)
+				(justify left bottom)
+			)
+		)
+		(property "Sheetfile" "DriversC.kicad_sch"
+			(at 224.155 48.8446 0)
+			(effects
+				(font
+					(size 1.27 1.27)
+				)
+				(justify left top)
+			)
+		)
+		(instances
+			(project "Nathophone_driver_board"
+				(path "/a109ba74-2574-4a03-88a2-446214ab2b70"
+					(page "6")
+				)
+			)
+		)
+	)
+	(sheet
+		(at 127.635 40.005)
+		(size 39.37 9.525)
+		(exclude_from_sim no)
+		(in_bom yes)
+		(on_board yes)
+		(dnp no)
+		(fields_autoplaced yes)
+		(stroke
+			(width 0.1524)
+			(type solid)
+		)
+		(fill
+			(color 0 0 0 0.0000)
+		)
+		(property "Sheetname" "Drivers A"
+			(at 127.635 39.2934 0)
+			(effects
+				(font
+					(size 1.27 1.27)
+				)
+				(justify left bottom)
+			)
+		)
+		(property "Sheetfile" "DriversA.kicad_sch"
+			(at 127.635 50.1146 0)
+			(effects
+				(font
+					(size 1.27 1.27)
+				)
+				(justify left top)
+			)
+		)
+		(instances
+			(project "Nathophone_driver_board"
+				(path "/a109ba74-2574-4a03-88a2-446214ab2b70"
+					(page "4")
+				)
+			)
+		)
+	)
+	(sheet
+		(at 83.185 38.735)
+		(size 32.385 9.525)
+		(exclude_from_sim no)
+		(in_bom yes)
+		(on_board yes)
+		(dnp no)
+		(fields_autoplaced yes)
+		(stroke
+			(width 0.1524)
+			(type solid)
+		)
+		(fill
+			(color 0 0 0 0.0000)
+		)
+		(property "Sheetname" "Data+Power Connections"
+			(at 83.185 38.0234 0)
+			(effects
+				(font
+					(size 1.27 1.27)
+				)
+				(justify left bottom)
+			)
+		)
+		(property "Sheetfile" "Nathophone_PCB_Data.kicad_sch"
+			(at 83.185 48.8446 0)
+			(effects
+				(font
+					(size 1.27 1.27)
+				)
+				(justify left top)
+			)
+		)
+		(instances
+			(project "Nathophone_driver_board"
+				(path "/a109ba74-2574-4a03-88a2-446214ab2b70"
+					(page "3")
+				)
+			)
+		)
+	)
+	(sheet
+		(at 178.435 39.37)
+		(size 39.37 10.795)
+		(exclude_from_sim no)
+		(in_bom yes)
+		(on_board yes)
+		(dnp no)
+		(fields_autoplaced yes)
+		(stroke
+			(width 0.1524)
+			(type solid)
+		)
+		(fill
+			(color 0 0 0 0.0000)
+		)
+		(property "Sheetname" "Drivers B"
+			(at 178.435 38.6584 0)
+			(effects
+				(font
+					(size 1.27 1.27)
+				)
+				(justify left bottom)
+			)
+		)
+		(property "Sheetfile" "DriversB.kicad_sch"
+			(at 178.435 50.7496 0)
+			(effects
+				(font
+					(size 1.27 1.27)
+				)
+				(justify left top)
+			)
+		)
+		(instances
+			(project "Nathophone_driver_board"
+				(path "/a109ba74-2574-4a03-88a2-446214ab2b70"
+					(page "5")
+				)
+			)
+		)
+	)
 	(sheet_instances
 		(path "/"
