File: pcb/DriversA.kicad_sch (KiCad schematic)
At the start: 49 parts, among them J13 54202-S0806ALF, J14 54202-S0806ALF, J5 TERM BLOCK, J6 TERM BLOCK, Q6 BSS84, Q7 BSS84, U3 TAS5720MRSMR, U4 TAS5720MRSMR

Commit message: ADDED Grounding Structure
Parts:
- U3, U4: footprint symbols_footprints:VQFN32_RSM0032B -> symbols_footprints:VQFN32_RSM0032B_NV
Changed lines of the file:
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@@
 			)
 		)
-		(property "Footprint" "symbols_footprints:VQFN32_RSM0032B"
+		(property "Footprint" "symbols_footprints:VQFN32_RSM0032B_NV"
 			(at 218.44 113.03 0)
 			(effects
@@
 			)
 		)
-		(property "Footprint" "symbols_footprints:VQFN32_RSM0032B"
+		(property "Footprint" "symbols_footprints:VQFN32_RSM0032B_NV"
 			(at 101.6 57.15 0)
 			(effects

Commit message: DONE Routing first two drivers
Connections:
- net ~{FAULT_0}: now also J14.12 (Pin_12); no longer J14.2 (Pin_2)
- net ~{FAULT_1}: now also J14.10 (Pin_10); no longer J14.4 (Pin_4)
- net ~{FAULT_2}: now also J14.8 (Pin_8); no longer J14.6 (Pin_6)
- net ~{FAULT_3}: now also J14.6 (Pin_6); no longer J14.8 (Pin_8)
- net ~{FAULT_4}: now also J14.4 (Pin_4); no longer J14.10 (Pin_10)
- net ~{FAULT_5}: now also J14.2 (Pin_2); no longer J14.12 (Pin_12)
Changed lines of the file:
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@@
 	(wire
 		(pts
+			(xy 99.06 137.16) (xy 101.6 137.16)
+		)
+		(stroke
+			(width 0)
+			(type default)
+		)
+	)
+	(wire
+		(pts
 			(xy 240.03 118.11) (xy 250.19 118.11)
 		)
@@
 	(wire
 		(pts
-			(xy 99.06 137.16) (xy 101.6 137.16)
-		)
-		(stroke
-			(width 0)
-			(type default)
-		)
-	)
-	(wire
-		(pts
 			(xy 124.46 85.09) (xy 124.46 90.17)
 		)
@@
 	(wire
 		(pts
+			(xy 99.06 124.46) (xy 101.6 124.46)
+		)
+		(stroke
+			(width 0)
+			(type default)
+		)
+	)
+	(wire
+		(pts
 			(xy 124.46 77.47) (xy 124.46 80.01)
 		)
@@
 	(wire
 		(pts
-			(xy 99.06 132.08) (xy 101.6 132.08)
-		)
-		(stroke
-			(width 0)
-			(type default)
-		)
-	)
-	(wire
-		(pts
 			(xy 240.03 107.95) (xy 240.03 105.41)
 		)
@@
 	(wire
 		(pts
-			(xy 99.06 134.62) (xy 101.6 134.62)
-		)
-		(stroke
-			(width 0)
-			(type default)
-		)
-	)
-	(wire
-		(pts
 			(xy 139.7 105.41) (xy 153.67 105.41)
 		)
@@
 	(wire
 		(pts
-			(xy 99.06 124.46) (xy 101.6 124.46)
-		)
-		(stroke
-			(width 0)
-			(type default)
-		)
-	)
-	(wire
-		(pts
 			(xy 43.18 163.83) (xy 43.18 157.48)
 		)
@@
 		)
 	)
-	(wire
+	(bus
 		(pts
-			(xy 99.06 129.54) (xy 101.6 129.54)
+			(xy 72.39 52.07) (xy 72.39 54.61)
 		)
 		(stroke
@@
 		)
 	)
-	(bus
+	(wire
 		(pts
-			(xy 72.39 52.07) (xy 72.39 54.61)
+			(xy 238.76 105.41) (xy 240.03 105.41)
 		)
 		(stroke
@@
 	(wire
 		(pts
-			(xy 238.76 105.41) (xy 240.03 105.41)
+			(xy 99.06 129.54) (xy 101.6 129.54)
 		)
 		(stroke
@@
 	(wire
 		(pts
+			(xy 99.06 127) (xy 101.6 127)
+		)
+		(stroke
+			(width 0)
+			(type default)
+		)
+	)
+	(wire
+		(pts
 			(xy 74.93 54.61) (xy 81.28 54.61)
 		)
@@
 	(wire
 		(pts
+			(xy 99.06 134.62) (xy 101.6 134.62)
+		)
+		(stroke
+			(width 0)
+			(type default)
+		)
+	)
+	(wire
+		(pts
 			(xy 241.3 128.27) (xy 241.3 133.35)
 		)
@@
 		)
 	)
+	(wire
+		(pts
+			(xy 99.06 132.08) (xy 101.6 132.08)
+		)
+		(stroke
+			(width 0)
+			(type default)
+		)
+	)
 	(bus
 		(pts
@@
 	(wire
 		(pts
-			(xy 99.06 127) (xy 101.6 127)
-		)
-		(stroke
-			(width 0)
-			(type default)
-		)
-	)
-	(wire
-		(pts
 			(xy 241.3 133.35) (xy 241.3 135.89)
 		)
@@
 	(global_label "~{FAULT_4}"
 		(shape input)
-		(at 101.6 134.62 0)
+		(at 101.6 127 0)
 		(fields_autoplaced yes)
 		(effects
@@
 		)
 		(property "Intersheetrefs" "${INTERSHEET_REFS}"
-			(at 111.7316 134.62 0)
+			(at 111.7316 127 0)
 			(effects
 				(font
@@
 	(global_label "~{FAULT_0}"
 		(shape input)
-		(at 101.6 124.46 0)
+		(at 101.6 137.16 0)
 		(fields_autoplaced yes)
 		(effects
@@
 		)
 		(property "Intersheetrefs" "${INTERSHEET_REFS}"
-			(at 111.7316 124.46 0)
+			(at 111.7316 137.16 0)
 			(effects
 				(font
@@
 	(global_label "~{FAULT_5}"
 		(shape input)
-		(at 101.6 137.16 0)
+		(at 101.6 124.46 0)
 		(fields_autoplaced yes)
 		(effects
@@
 		)
 		(property "Intersheetrefs" "${INTERSHEET_REFS}"
-			(at 111.7316 137.16 0)
+			(at 111.7316 124.46 0)
 			(effects
 				(font
@@
 	(global_label "~{FAULT_2}"
 		(shape input)
-		(at 101.6 129.54 0)
+		(at 101.6 132.08 0)
 		(fields_autoplaced yes)
 		(effects
@@
 		)
 		(property "Intersheetrefs" "${INTERSHEET_REFS}"
-			(at 111.7316 129.54 0)
+			(at 111.7316 132.08 0)
 			(effects
 				(font
@@
 	(global_label "~{FAULT_1}"
 		(shape input)
-		(at 101.6 127 0)
+		(at 101.6 134.62 0)
 		(fields_autoplaced yes)
 		(effects
@@
 		)
 		(property "Intersheetrefs" "${INTERSHEET_REFS}"
-			(at 111.7316 127 0)
+			(at 111.7316 134.62 0)
 			(effects
 				(font
@@
 	(global_label "~{FAULT_3}"
 		(shape input)
-		(at 101.6 132.08 0)
+		(at 101.6 129.54 0)
 		(fields_autoplaced yes)
 		(effects
@@
 		)
 		(property "Intersheetrefs" "${INTERSHEET_REFS}"
-			(at 111.7316 132.08 0)
+			(at 111.7316 129.54 0)
 			(effects
 				(font

Commit message: DONE Digital Routing
Connections:
- net at C25.2, L5.2, R15.1: now also J5.1 (Pin_1), J5.2 (Pin_2); no longer J5.3 (Pin_3), J5.4 (Pin_4)
- net at C31.2, L7.2, R19.1: now also J6.1 (Pin_1), J6.2 (Pin_2); no longer J6.3 (Pin_3), J6.4 (Pin_4)
- net at C24.1, L4.2, R14.2: now also J5.3 (Pin_3), J5.4 (Pin_4); no longer J5.1 (Pin_1), J5.2 (Pin_2)
- net at C30.1, L6.2, R18.2: now also J6.3 (Pin_3), J6.4 (Pin_4); no longer J6.1 (Pin_1), J6.2 (Pin_2)

Commit message: CHANGED small things, removed tiny 0201 cap
Parts:
- C19, C21, C32, C35: MPN (none) -> GRM3195C1H104JA05D
- C20, C22, C33, C36: MPN (none) -> A782MS107M1JLAS030
- C23, C26, C29, C34, C37, C38, C41, C42: MPN (none) -> CL21B105KAFNNNE
- C24, C25, C30, C31: MPN (none) -> SMDTC03680QB00MP00
- C27, C28, C39, C40: MPN (none) -> GRM31C5C1H224JE02L
- D4, D5: MPN (none) -> CMD17-21VRD/TR8
- J13, J14: MPN (none) -> 54202-S0806ALF
- J5, J6: MPN (none) -> 1862042
- L3: MPN (none) -> 74404086151
- L4, L5, L6, L7: MPN (none) -> SRU1048-150Y
- Q6, Q7: MPN (none) -> BSS84
- R14, R15, R18, R19: MPN (none) -> CRCW20100000Z0EF
- R16, R20: MPN (none) -> CRCW08051K00FKEA
- R17, R21: MPN (none) -> CRCW0805100KFKEA
- R22: MPN (none) -> CRCW080522K0FKEB
- U3, U4: MPN (none) -> TAS5720MRSMR

Commit message: SIMULATED Transmission line, LAST checks, ORDERED pcb
Parts:
- renumbered C19 to C22, C20 to C23, C21 to C24, C22 to C25, C23 to C26, C24 to C27, C25 to C28, C26 to C29, C27 to C30, C28 to C31, C29 to C32, C30 to C33, C31 to C34, C32 to C35, C33 to C36, C34 to C37, C35 to C38, C36 to C39, C37 to C40, C38 to C41, C39 to C42, C40 to C43, C41 to C44, C42 to C45, D4 to D6, D5 to D7, J13 to J6, J5 to J7, J14 to J8, J6 to J9, Q6 to Q8, Q7 to Q9, R14 to R25, R15 to R26, R16 to R27, R17 to R28, R18 to R29, R19 to R30, R20 to R31, R21 to R32, R22 to R33, TP8 to TP7, U3 to U4, U4 to U5
Connections:
- net DATA renamed DATA_B
- net LRCLK renamed LRCLK_B
- net MRCLK renamed MRCLK_B
- net SCLK renamed SCLK_B
