File: pcb/DriversB.kicad_sch (KiCad schematic)
At the start: 47 parts, among them J7 TERM BLOCK, J8 TERM BLOCK, Q8 BSS84, Q9 BSS84, U5 TAS5720MRSMR, U6 TAS5720MRSMR

Commit message: ADDED Grounding Structure
Parts:
- U5, U6: footprint symbols_footprints:VQFN32_RSM0032B -> symbols_footprints:VQFN32_RSM0032B_NV
Changed lines of the file:
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@@
 			)
 		)
-		(property "Footprint" "symbols_footprints:VQFN32_RSM0032B"
+		(property "Footprint" "symbols_footprints:VQFN32_RSM0032B_NV"
 			(at 218.44 113.03 0)
 			(effects
@@
 			)
 		)
-		(property "Footprint" "symbols_footprints:VQFN32_RSM0032B"
+		(property "Footprint" "symbols_footprints:VQFN32_RSM0032B_NV"
 			(at 101.6 57.15 0)
 			(effects

Commit message: DONE Routing first two drivers
Connections:
- net OUT1_N is gone; now on net OUT3_N: C52.2, U5.16 (OUT_N), U5.17 (OUT_N)
- net OUT1_P is gone; now on net OUT3_P: C51.2, U5.24 (OUT_P), U5.25 (OUT_P)
- net OUT2_N is gone; now on net OUT4_N: C64.2, U6.16 (OUT_N), U6.17 (OUT_N)
- net OUT2_P is gone; now on net OUT4_P: C63.2, U6.24 (OUT_P), U6.25 (OUT_P)
Changed lines of the file:
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@@
 		)
 	)
-	(label "OUT1_P"
+	(label "OUT3_P"
 		(at 138.43 44.45 0)
 		(effects
@@
 		)
 	)
-	(label "OUT2_P"
+	(label "OUT4_P"
 		(at 251.46 100.33 0)
 		(effects
@@
 		)
 	)
-	(label "OUT2_N"
+	(label "OUT4_N"
 		(at 251.46 118.11 0)
 		(effects
@@
 		)
 	)
-	(label "OUT1_N"
+	(label "OUT3_N"
 		(at 138.43 57.15 0)
 		(effects

Commit message: DONE Digital Routing
Connections:
- net at C54.1, L11.2, R28.2: now also J8.3 (Pin_3), J8.4 (Pin_4); no longer J8.1 (Pin_1), J8.2 (Pin_2)
- net at C55.2, L12.2, R29.1: now also J8.1 (Pin_1), J8.2 (Pin_2); no longer J8.3 (Pin_3), J8.4 (Pin_4)
- net at C49.2, L10.2, R24.1: now also J7.1 (Pin_1), J7.2 (Pin_2); no longer J7.3 (Pin_3), J7.4 (Pin_4)
- net at C48.1, L9.2, R23.2: now also J7.3 (Pin_3), J7.4 (Pin_4); no longer J7.1 (Pin_1), J7.2 (Pin_2)

Commit message: CHANGED small things, removed tiny 0201 cap
Parts:
- C43, C45, C56, C59: MPN (none) -> GRM3195C1H104JA05D
- C44, C46, C57, C60: MPN (none) -> A782MS107M1JLAS030
- C47, C50, C53, C58, C61, C62, C65, C66: MPN (none) -> CL21B105KAFNNNE
- C48, C49, C54, C55: MPN (none) -> SMDTC03680QB00MP00
- C51, C52, C63, C64: MPN (none) -> GRM31C5C1H224JE02L
- D6, D7: MPN (none) -> CMD17-21VRD/TR8
- J7, J8: MPN (none) -> 1862042
- L10, L11, L12, L9: MPN (none) -> SRU1048-150Y
- L8: MPN (none) -> 74404086151
- Q8, Q9: MPN (none) -> BSS84
- R23, R24, R28, R29: MPN (none) -> CRCW20100000Z0EF
- R25, R30: MPN (none) -> CRCW08051K00FKEA
- R26, R31: MPN (none) -> CRCW0805100KFKEA
- R27: MPN (none) -> CRCW080522K0FKEB
- U5, U6: MPN (none) -> TAS5720MRSMR

Commit message: SIMULATED Transmission line, LAST checks, ORDERED pcb
Parts:
- added R39, R40, R41, R42: 40R2, Resistor_SMD:R_0805_2012Metric, symbol Device:R
- renumbered C43 to C46, C44 to C47, C45 to C48, C46 to C49, C47 to C50, C48 to C51, C49 to C52, C50 to C53, C51 to C54, C52 to C55, C53 to C56, C54 to C57, C55 to C58, C56 to C59, C57 to C60, C58 to C61, C59 to C62, C60 to C63, C61 to C64, C62 to C65, C63 to C66, C64 to C67, C65 to C68, C66 to C69, D6 to D8, D7 to D9, J7 to J10, J8 to J11, Q8 to Q10, Q9 to Q11, R23 to R34, R24 to R35, R25 to R36, R26 to R37, R27 to R38, R28 to R43, R29 to R44, R30 to R45, R31 to R46, TP9 to TP8, U5 to U6, U6 to U7
Connections:
- net DATA renamed DATA_A
- net DATA_A: now also R42.2; no longer U6.7 (SDIN)
- net LRCLK renamed LRCLK_A
- net LRCLK_A: now also R41.1; no longer U6.4 (LRCLK)
- net MRCLK renamed MRCLK_A
- net MRCLK_A: now also R39.1; no longer U6.5 (MCLK)
- net SCLK renamed SCLK_A
- net SCLK_A: now also R40.2; no longer U6.6 (BCLK)
- new net DATA_B: R42.1, U6.7 (SDIN)
- new net LRCLK_B: R41.2, U6.4 (LRCLK)
- new net MRCLK_B: R39.2, U6.5 (MCLK)
- new net SCLK_B: R40.1, U6.6 (BCLK)
