File: pcb/DriversC.kicad_sch (KiCad schematic)
At the start: 49 parts, among them J10 TERM BLOCK, J9 TERM BLOCK, Q10 BSS84, Q11 BSS84, U7 TAS5720MRSMR, U8 TAS5720MRSMR

Commit message: ADDED Grounding Structure
Parts:
- U7, U8: footprint symbols_footprints:VQFN32_RSM0032B -> symbols_footprints:VQFN32_RSM0032B_NV
Changed lines of the file:
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@@
 			)
 		)
-		(property "Footprint" "symbols_footprints:VQFN32_RSM0032B"
+		(property "Footprint" "symbols_footprints:VQFN32_RSM0032B_NV"
 			(at 218.44 113.03 0)
 			(effects
@@
 			)
 		)
-		(property "Footprint" "symbols_footprints:VQFN32_RSM0032B"
+		(property "Footprint" "symbols_footprints:VQFN32_RSM0032B_NV"
 			(at 101.6 57.15 0)
 			(effects

Commit message: DONE Routing first two drivers
Connections:
- net OUT1_N is gone; now on net OUT5_N: C76.2, U7.16 (OUT_N), U7.17 (OUT_N)
- net OUT1_P is gone; now on net OUT5_P: C75.2, U7.24 (OUT_P), U7.25 (OUT_P)
- net OUT2_N is gone; now on net OUT6_N: C88.2, U8.16 (OUT_N), U8.17 (OUT_N)
- net OUT2_P is gone; now on net OUT6_P: C87.2, U8.24 (OUT_P), U8.25 (OUT_P)
Changed lines of the file:
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@@
 		)
 	)
-	(label "OUT1_P"
+	(label "OUT5_P"
 		(at 138.43 44.45 0)
 		(effects
@@
 		)
 	)
-	(label "OUT1_N"
+	(label "OUT5_N"
 		(at 138.43 57.15 0)
 		(effects
@@
 		)
 	)
-	(label "OUT2_P"
+	(label "OUT6_P"
 		(at 251.46 100.33 0)
 		(effects
@@
 		)
 	)
-	(label "OUT2_N"
+	(label "OUT6_N"
 		(at 251.46 118.11 0)
 		(effects

Commit message: DONE Digital Routing
Connections:
- net at C78.1, L16.2, R37.2: now also J10.3 (Pin_3), J10.4 (Pin_4); no longer J10.1 (Pin_1), J10.2 (Pin_2)
- net at C73.2, L15.2, R33.1: now also J9.1 (Pin_1), J9.2 (Pin_2); no longer J9.3 (Pin_3), J9.4 (Pin_4)
- net at C72.1, L14.2, R32.2: now also J9.3 (Pin_3), J9.4 (Pin_4); no longer J9.1 (Pin_1), J9.2 (Pin_2)
- net at C79.2, L17.2, R38.1: now also J10.1 (Pin_1), J10.2 (Pin_2); no longer J10.3 (Pin_3), J10.4 (Pin_4)

Commit message: CHANGED small things, removed tiny 0201 cap
Parts:
- C67, C69, C80, C83: MPN (none) -> GRM3195C1H104JA05D
- C68, C70, C81, C84: MPN (none) -> A782MS107M1JLAS030
- C71, C74, C77, C82, C85, C86, C89, C90: MPN (none) -> CL21B105KAFNNNE
- C72, C73, C78, C79: MPN (none) -> SMDTC03680QB00MP00
- C75, C76, C87, C88: MPN (none) -> GRM31C5C1H224JE02L
- D8, D9: MPN (none) -> CMD17-21VRD/TR8
- J10, J9: MPN (none) -> 1862042
- L13: MPN (none) -> 74404086151
- L14, L15, L16, L17: MPN (none) -> SRU1048-150Y
- Q10, Q11: MPN (none) -> BSS84
- R32, R33, R37, R38: MPN (none) -> CRCW20100000Z0EF
- R34, R39: MPN (none) -> CRCW08051K00FKEA
- R35, R40: MPN (none) -> CRCW0805100KFKEA
- R36, R41, R42: MPN (none) -> CRCW080522K0FKEB
- U7, U8: MPN (none) -> TAS5720MRSMR

Commit message: SIMULATED Transmission line, LAST checks, ORDERED pcb
Parts:
- renumbered C67 to C70, C68 to C71, C69 to C72, C70 to C73, C71 to C74, C72 to C75, C73 to C76, C74 to C77, C75 to C78, C76 to C79, C77 to C80, C78 to C81, C79 to C82, C80 to C83, C81 to C84, C82 to C85, C83 to C86, C84 to C87, C85 to C88, C86 to C89, C87 to C90, C88 to C91, C89 to C92, C90 to C93, D8 to D10, D9 to D11, J9 to J12, J10 to J13, Q10 to Q12, Q11 to Q13, R32 to R47, R33 to R48, R34 to R49, R35 to R50, R36 to R51, R37 to R52, R38 to R53, R39 to R54, R40 to R55, R41 to R56, R42 to R57, TP10 to TP9, U7 to U8, U8 to U9
Connections:
- net DATA renamed DATA_A
- net LRCLK renamed LRCLK_A
- net MRCLK renamed MRCLK_A
- net SCLK renamed SCLK_A
