File: pcb/Nathophone_PCB_Data.kicad_sch (KiCad schematic)
At the start: 23 parts, among them J11 54202-S0806ALF, J3 Conn_01x30, J4 54202-S0806ALF, Q12 2N7002H, Q13 2N7002H, SW2 PTS645SM43SMTR92 LFS, SW3 DS04-254-2-01BK-SMT, U10 74LVC2G07

Commit message: FINISHED Version 1, Checked heights
Parts:
- added F1, F2: Polyfuse, Fuse:Fuse_1812_4532Metric, symbol Device:Polyfuse
- added F3, F4: Polyfuse, Fuse:Fuse_1206_3216Metric, symbol Device:Polyfuse
Connections:
- net +3.3V_ext: now also F3.1; no longer J11.2 (Pin_2)
- net +3.3V_int: now also F1.1; no longer J4.5 (Pin_5), J4.7 (Pin_7)
- net +5.3V: now also F2.1; no longer D12.2 (A)
- net +5V_ext: now also F4.1; no longer J11.4 (Pin_4)
- new net: F4.2, J11.4 (Pin_4)
- new net: F3.2, J11.2 (Pin_2)
- new net: F1.2, J4.5 (Pin_5), J4.7 (Pin_7)
- new net: D12.2 (A), F2.2

Commit message: CHANGED small things, removed tiny 0201 cap
Parts:
- C18, C92: MPN (none) -> CL21C103JBF1PNE
- C91: MPN (none) -> GRM3195C1H104JA05D
- D10: MPN (none) -> CMD15-21VYD/TR8
- D12, D3: MPN (none) -> SL215B-TP
- F1, F2: MPN (none) -> MINISMDC125F-2
- F3, F4: MPN (none) -> 0ZCJ0025AF2E
- J11, J4: MPN (none) -> 54202-S0806ALF
- J3: MPN (none) -> 0525593072
- Q12, Q13: MPN (none) -> 2N7002H-7
- R13, R45, R47: MPN (none) -> CRCW0805100KFKEA
- R43: MPN (none) -> CRCW0805470RJNEA
- SW2: MPN (none) -> PTS645SM43SMTR92 LFS
- SW3: MPN (none) -> DS04-254-2-01BK-SMT
- U10: MPN (none) -> SN74LVC2G07DCKR

Commit message: SIMULATED Transmission line, LAST checks, ORDERED pcb
Parts:
- removed D12: SL215B-TP, Diode_SMD:D_SMB, symbol Diode:B220
- added R19, R20, R21, R22: 40R2, Resistor_SMD:R_0805_2012Metric, symbol Device:R
- added R23, R24: 3k, Resistor_SMD:R_0805_2012Metric, symbol Device:R
- renumbered C18 to C19, C92 to C20, C91 to C21, D10 to D4, D3 to D5, F1 to F4, F2 to F5, F3 to F6, F4 to F7, J11 to J5, Q12 to Q6, Q13 to Q7, R43 to R15, R45 to R16, R47 to R17, R13 to R18, TP1 to TP2, TP2 to TP3, TP3 to TP4, TP4 to TP5, TP5 to TP6, U10 to U3
Connections:
- net +3.3V_int: now also R23.1, R24.1
- net SCL: now also R23.2
- net SDA: now also R24.2
- net at J4.1 (Pin_1), J4.3 (Pin_3): now also F5.2
- net DATA renamed DATA_IN
- net DATA_IN: now also R19.1
- net LRCLK renamed LRCLK_IN
- net LRCLK_IN: now also R21.1
- net MRCLK renamed MRCLK_IN
- net MRCLK_IN: now also R22.2
- net SCLK renamed SCLK_IN
- net SCLK_IN: now also R20.2
- new net DATA_A: R19.2
- new net LRCLK_A: R21.2
- new net MRCLK_A: R22.1
- new net SCLK_A: R20.1
Other:
- note added: "33R Resistors provided on Milan Board"
- note added: "Pull-ups provided on Milan Board"
- note removed: "Pull-ups provided on board"
- moved on the sheet: F4, F5, J4, TP4
