File: USBtoI2S_board/nathophone_USBtoI2S/Connectors_Power_Misc.kicad_sch (KiCad schematic)
At the start: 42 parts, among them J1 UJ20-C-H-G-SMT-5-P16-TR, J2 FTSH-110-01-F-DV-K, J3 Conn_01x30, J4 FTSH-105-01-F-DV-P-TR, Q1 MMBT3904, SW1 PEC09-2320F-S0015, U1 IS25LP032D-JKLE

Commit message: PLACED all footprints and GND zone
Parts:
- removed TP10, TP11, TP12, TP7, TP9: TestPoint_Small, TestPoint:TestPoint_Pad_D1.5mm, symbol Connector:TestPoint_Small
Connections:
- net ~{~{VBUS_DET}} renamed ~{VBUS_DET}
Other:
- note added: "Aux/Test Connector"
- moved on the sheet: C37, C38, C39, J4, R24, R25, R26, SW1
