File: USBtoI2S_board/nathophone_USBtoI2S/Connectors_Power_Misc.kicad_sch (KiCad schematic)
At the start: 37 parts, among them J1 UJ20-C-H-G-SMT-5-P16-TR, J2 FTSH-110-01-F-DV-K, J3 Conn_01x30, J4 FTSH-105-01-F-DV-P-TR, Q1 MMBT3904, SW1 PEC09-2320F-S0015, U1 IS25LP032D-JKLE

Commit message: ADDED USBtoI2S board design files
Parts:
- added D1: 5.6V, USB_to_I2S_Board:SOD-962_SL2_TOS, symbol Device:D_TVS_Small
Connections:
- net +5V: now also D1.2 (A2)
- net GND: now also D1.1 (A1)
Other:
- title: USB to I2S Module -> Nathophone USB_to_I2S Module
