File: USBtoI2S_board/nathophone_USBtoI2S/Power.kicad_sch (KiCad schematic)
At the start: 23 parts, among them U3 TPS62410DRCR, U4 MAX809STRG, U5 74LVC2G07

Commit message: PLACED all footprints and GND zone
Parts:
- removed TP4: TestPoint_Small, TestPoint:TestPoint_Pad_D1.5mm, symbol Connector:TestPoint_Small
Other:
- moved on the sheet: R23, TP13, TP5, U5A, U5B
