File: USBtoI2S_board/nathophone_USBtoI2S/Power.kicad_sch (KiCad schematic)
At the start: 22 parts, among them U3 TPS62410DRCR, U4 MAX809STRG, U5 74LVC2G07

Commit message: ADDED USBtoI2S board design files
Parts:
- added C42, C43: 10u, Capacitor_SMD:C_1210_3225Metric_Pad1.33x2.70mm_HandSolder, symbol Device:C_Small
- added U6: AP7361C-33FGE-7, USB_to_I2S_Board:SON65P300X300X63-9N, symbol USB_to_I2S_Board:AP7361C-FGE-7
Connections:
- net +3.3V: now also C43.1, U6.1 (OUT)
- net +5V: now also C42.1, U6.5 (EN), U6.8 (IN)
- net GND: now also C42.2, C43.2, U6.4 (GND), U6.9 (GND__1)
Other:
- company: (none) -> Private
- title: (none) -> Nathophone USB_to_I2S Module
