File: USBtoI2S_board/nathophone_USBtoI2S/xmos.kicad_sch (KiCad schematic)
At the start: 17 parts, among them U2 XU316-1024-TQ128-C24, Y1 FA-238 24MHz

Commit message: ADDED XMOS eval board design files, BEGUN layout of usbtoi2s board
Parts:
- added C10, C11, C12, C13, C18, C19, C20, C21, C22, C23, C24, C25, C26, C27, C28, C29, C30, C31, C32, C33, C35, C36, C41: 100n, USB_to_I2S_Board:CAPC1810X65N, symbol Device:C_Small
- added C34: 1u, Capacitor_SMD:C_0603_1608Metric, symbol Device:C_Small
- added C40: 2.2u, Capacitor_SMD:C_0805_2012Metric_Pad1.18x1.45mm_HandSolder, symbol Device:C_Small
- added D1: LTST-C235KGKRKT, LED_SMD:LED_LiteOn_LTST-C235KGKRKT, symbol LED:LTST-C235KGKRKT
- added FB1: 600R @ 100MHz, Capacitor_SMD:C_0805_2012Metric_Pad1.18x1.45mm_HandSolder, symbol Device:FerriteBead_Small
- added R27: 113R, Resistor_SMD:R_0805_2012Metric_Pad1.20x1.40mm_HandSolder, symbol Device:R_Small
- added R28: 147R, Resistor_SMD:R_0805_2012Metric_Pad1.20x1.40mm_HandSolder, symbol Device:R_Small
- renumbered C7 to C6, C6 to C7, R17 to R10, R7 to R11, R14 to R12, R15 to R13, R16 to R14, R11 to R15, R12 to R16, R13 to R17, R18 to R8, R8 to R9
Connections:
- net +3.3V: now also U2.10 (VDDIOL), U2.109 (VDDIOT), U2.121 (VDDIOT__1), U2.17 (VDDIOL__1), U2.61 (USB_VDD33), U2.72 (VDDIOR), U2.89 (VDDIOR__1), C26.1, C27.1, C28.1, C29.1, C30.1, C31.1, C36.1
- net GND: now also U2.129 (VSS__1), U2.24 (MIPI_VDD18), U2.27 (MIPI_VDD09), U2.30 (VSS), U2.42 (PLL_AGND), C10.2, C11.2, C12.2, C13.2, C18.2, C19.2, C20.2, C21.2, C22.2, C23.2, C24.2, C25.2, C26.2, C27.2, C28.2, C29.2, C30.2, C31.2, C32.2, C33.2, C34.2, C35.2, C36.2, C40.2, C41.2, D1.1 (K2), D1.4 (K1)
- net VDD: now reaches U2.104 (VDD__11)
- net VDD: now also U2.105 (VDD__12), U2.106 (VDD__13), U2.11 (VDD__1), U2.113 (VDD__14), U2.14 (VDD__2), U2.18 (VDD__3), U2.39 (VDD__4), U2.45 (VDD__5), U2.5 (VDD), U2.50 (VDD__6), U2.54 (VDD__7), U2.68 (VDD__8), U2.85 (VDD__9), U2.95 (VDD__10), C10.1, C11.1, C12.1, C13.1, C18.1, C19.1, C20.1, C21.1, C22.1, C23.1, C24.1, C25.1, C40.1, C41.1, FB1.1
- net +1V8: now reaches U2.35 (VDDIOB18)
- net +1V8: now also U2.56 (VDDIOB18__1), U2.62 (USB_VDD18), C32.1, C33.1, C35.1
- net ~{SYS_RESET}: now reaches U2.38 (~{RST})
- net at U2.41 (PLL_AVDD): now also C34.1, FB1.2
- net at U2.79 (X1D53): now also R28.1
- net at U2.80 (X1D54): now also R27.2
- net GPIO: now reaches U2.81 (X1D55)
- net Rot_Enc_A: now reaches U2.82 (X1D56)
- net Rot_Enc_B: now reaches U2.83 (X1D57)
- net Rot_Enc_SW: now reaches U2.84 (X1D58)
- new net: D1.2 (A2), R27.1
- new net: D1.3 (A1), R28.2
Other:
- moved on the sheet: C6, C7, JP1, R10, R11, R12, R13, R14, R15, R16, R17, R8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

Commit message: PLACED all footprints and GND zone
Parts:
- removed D1: LTST-C235KGKRKT, LED_SMD:LED_LiteOn_LTST-C235KGKRKT, symbol LED:LTST-C235KGKRKT
- added D2: XZMDKVG55W-8, USB_to_I2S_Board:LED_XZMDKVG55W-8, symbol Device:LED_Dual_AKAK
- R27: value 113R -> 750R; DigiKey Part Number 541-113CCT-ND -> 541-750CCT-ND; MPN CRCW0805113RFKEA -> CRCW0805750RFKEA; Tol. 0.5% -> 1%
- R28: value 147R -> 680R; DigiKey Part Number 541-147CCT-ND -> 541-680CCT-ND; MPN CRCW0805147RFKEA -> CRCW0805680RFKEA; Tol. 0.5% -> 1%
Connections:
- net GND: now also D2.2 (K1), D2.4 (K2)
- net at R27.1: now also D2.3 (A2)
- net at R28.2: now also D2.1 (A1)
Other:
- note added: "GN"
- note added: "RD"
