File: USBtoI2S_board/nathophone_USBtoI2S/xmos.kicad_sch (KiCad schematic)
At the start: 46 parts, among them U2 XU316-1024-TQ128-C24, Y1 FA-238 24MHz

Commit message: ADDED USBtoI2S board design files
Other:
- title: USB to I2S Module -> Nathophone USB_to_I2S Module
Changed lines of the file:
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@@
 	(paper "A4")
 	(title_block
-		(title "USB to I2S Module")
-		(date "2026-05-07")
-		(rev "0")
+		(title "Nathophone USB_to_I2S Module")
+		(date "2026-08-08")
+		(rev "v3")
 		(company "Private")
 	)
@@
 			)
 		)
-		(property "Datasheet" "https://www.xmos.com/documentation/XM-014532-PC/pdf/XU316-1024-TQ128.pdf"
+		(property "Datasheet" "https://www.xmos.com/documentation/XM-014532-PC/html/rst/XU316-1024-TQ128.html"
 			(at 82.55 90.17 0)
 			(hide yes)
