File: USBtoI2S_board/nathophone_USBtoI2S/nathophone_USBtoI2S.kicad_pcb (KiCad board)
At the start: 2 copper layers, 80 x 40 mm, 9 parts, among them J1 Conn_01x30, J2 UJ20-C-H-G-SMT-5-P16-TR

Commit message: ADDED XMOS eval board design files, BEGUN layout of usbtoi2s board
Parts:
- removed ? (x4): , 
- added C1: 100n, USB_to_I2S_Board:CAPC1810X65N, F.Cu at (111.3, 96.9)
- added C10: 100n, USB_to_I2S_Board:CAPC1810X65N, F.Cu at (347.5, 2.08)
- added C11: 100n, USB_to_I2S_Board:CAPC1810X65N, F.Cu at (347.5, 7.67)
- added C12: 100n, USB_to_I2S_Board:CAPC1810X65N, F.Cu at (359.8, -6.41)
- added C13: 100n, USB_to_I2S_Board:CAPC1810X65N, F.Cu at (372.4, -4.01)
- added C14: 22p, Capacitor_SMD:C_0603_1608Metric_Pad1.08x0.95mm_HandSolder, F.Cu at (443.6, -5.08)
- added C15: 22u, Capacitor_SMD:C_1210_3225Metric_Pad1.33x2.70mm_HandSolder, F.Cu at (455.2, 3.81)
- added C16: 22u, Capacitor_SMD:C_1210_3225Metric_Pad1.33x2.70mm_HandSolder, F.Cu at (455.2, -0.76)
- added C17: 10u, Capacitor_SMD:C_1210_3225Metric_Pad1.33x2.70mm_HandSolder, F.Cu at (439.9, 1.27)
- added C18: 100n, USB_to_I2S_Board:CAPC1810X65N, F.Cu at (372.4, 3.61)
- added C19: 100n, USB_to_I2S_Board:CAPC1810X65N, F.Cu at (372.6, 12.8)
- added C2: 100n, USB_to_I2S_Board:CAPC1810X65N, F.Cu at (227.5, 62.8)
- added C20: 100n, USB_to_I2S_Board:CAPC1810X65N, F.Cu at (365.7, -6.41)
- added C21: 100n, USB_to_I2S_Board:CAPC1810X65N, F.Cu at (347.5, 3.86)
- added C22: 100n, USB_to_I2S_Board:CAPC1810X65N, F.Cu at (356.3, 17.4)
- added C23: 100n, USB_to_I2S_Board:CAPC1810X65N, F.Cu at (363.9, 17.4)
- added C24: 100n, USB_to_I2S_Board:CAPC1810X65N, F.Cu at (362.1, 17.4)
- added C25: 100n, USB_to_I2S_Board:CAPC1810X65N, F.Cu at (360.3, 17.4)
- added C26: 100n, USB_to_I2S_Board:CAPC1810X65N, F.Cu at (372.4, 1.83)
- added C27: 100n, USB_to_I2S_Board:CAPC1810X65N, F.Cu at (372.6, 6.91)
- added C28: 100n, USB_to_I2S_Board:CAPC1810X65N, F.Cu at (356.8, -6.41)
- added C29: 100n, USB_to_I2S_Board:CAPC1810X65N, F.Cu at (361.6, -6.41)
- added C3: 100n, USB_to_I2S_Board:CAPC1810X65N, F.Cu at (227.5, 65.5)
- added C30: 100n, USB_to_I2S_Board:CAPC1810X65N, F.Cu at (347.5, 0.30)
- added C31: 100n, USB_to_I2S_Board:CAPC1810X65N, F.Cu at (347.5, 5.89)
- added C32: 100n, USB_to_I2S_Board:CAPC1810X65N, F.Cu at (365.7, 17.4)
- added C33: 100n, USB_to_I2S_Board:CAPC1810X65N, F.Cu at (354.5, 17.4)
- added C34: 1u, Capacitor_SMD:C_0603_1608Metric, F.Cu at (357.6, 15.0)
- added C35: 100n, USB_to_I2S_Board:CAPC1810X65N, F.Cu at (369.2, 17.4)
- added C36: 100n, USB_to_I2S_Board:CAPC1810X65N, F.Cu at (367.5, 17.4)
- added C37: 10n, Capacitor_SMD:C_0805_2012Metric_Pad1.18x1.45mm_HandSolder, F.Cu at (223.0, 63.3)
- added C38: 10n, Capacitor_SMD:C_0805_2012Metric_Pad1.18x1.45mm_HandSolder, F.Cu at (223.0, 66.3)
- added C39: 10n, Capacitor_SMD:C_0805_2012Metric_Pad1.18x1.45mm_HandSolder, F.Cu at (223.0, 69.3)
- added C4: 10n, Capacitor_SMD:C_0805_2012Metric_Pad1.18x1.45mm_HandSolder, F.Cu at (223.0, 60.3)
- added C40: 2.2u, Capacitor_SMD:C_0805_2012Metric_Pad1.18x1.45mm_HandSolder, F.Cu at (363.6, -6.58)
- added C41: 100n, USB_to_I2S_Board:CAPC1810X65N, F.Cu at (347.5, -1.47)
- added C5: 100n, USB_to_I2S_Board:CAPC1810X65N, F.Cu at (227.5, 68.2)
- added C6: 18p, Capacitor_SMD:C_0603_1608Metric, F.Cu at (346.1, 18.0)
- added C7: 18p, Capacitor_SMD:C_0603_1608Metric, F.Cu at (352.5, 18.0)
- added C8: 100n, USB_to_I2S_Board:CAPC1810X65N, F.Cu at (243.6, 79.2)
- added C9: 100n, USB_to_I2S_Board:CAPC1810X65N, F.Cu at (243.6, 81.9)
- added D1: LTST-C235KGKRKT, LED_SMD:LED_LiteOn_LTST-C235KGKRKT, F.Cu at (260.9, 56.4)
- added FB1: 600R @ 100MHz, Capacitor_SMD:C_0805_2012Metric_Pad1.18x1.45mm_HandSolder, F.Cu at (358.3, 17.9)
- added H1: MountingHole, MountingHole:MountingHole_2.7mm_M2.5_DIN965, F.Cu at (222.1, 110.3)
- added H2: MountingHole, MountingHole:MountingHole_2.7mm_M2.5_DIN965, F.Cu at (222.1, 116.6)
- added H3: MountingHole, MountingHole:MountingHole_2.7mm_M2.5_DIN965, F.Cu at (222.1, 122.8)
- added H4: MountingHole, MountingHole:MountingHole_2.7mm_M2.5_DIN965, F.Cu at (222.1, 129.1)
- added J3: Conn_01x30, Nathophone_Driverboard:CON_525593072_MOL, F.Cu at (201.3, 90.2)
- added J4: FTSH-105-01-F-DV-P-TR, Connector_PinHeader_1.27mm:PinHeader_2x05_P1.27mm_Vertical_SMD, F.Cu at (228.9, 32.9)
- added JP1: SolderJumper_2_Open, Jumper:SolderJumper-2_P1.3mm_Open_RoundedPad1.0x1.5mm, F.Cu at (342.9, 13.5)
- added L1: 2.2uH, USB_to_I2S_Board:IND_EPCOS_B82432T_EPC, F.Cu at (449.4, 3.81)
- added L2: 3.3uH, USB_to_I2S_Board:IND_EPCOS_B82432T_EPC, F.Cu at (449.4, -0.76)
- added Q1: MMBT3904, Package_TO_SOT_SMD:SOT-23, F.Cu at (228.9, 42.0)
- added R10: 1M, Resistor_SMD:R_0603_1608Metric, F.Cu at (351.6, 15.3)
- added R11: 4k7, Resistor_SMD:R_0805_2012Metric_Pad1.20x1.40mm_HandSolder, F.Cu at (372.5, 0.05)
- added R12: 33R, Resistor_SMD:R_0805_2012Metric_Pad1.20x1.40mm_HandSolder, F.Cu at (372.8, 10.7)
- added R13: 33R, Resistor_SMD:R_0805_2012Metric_Pad1.20x1.40mm_HandSolder, F.Cu at (372.8, 8.69)
- added R14: 33R, Resistor_SMD:R_0805_2012Metric_Pad1.20x1.40mm_HandSolder, F.Cu at (340.8, 4.88)
- added R15: 33R, Resistor_SMD:R_0805_2012Metric_Pad1.20x1.40mm_HandSolder, F.Cu at (340.8, 6.91)
- added R16: 33R, Resistor_SMD:R_0805_2012Metric_Pad1.20x1.40mm_HandSolder, F.Cu at (347.4, 9.70)
- added R17: 33R, Resistor_SMD:R_0805_2012Metric_Pad1.20x1.40mm_HandSolder, F.Cu at (347.4, 11.7)
- added R18: 100k, Resistor_SMD:R_0805_2012Metric_Pad1.20x1.40mm_HandSolder, F.Cu at (443.5, 6.35)
- added R19: 200k, Resistor_SMD:R_0805_2012Metric_Pad1.20x1.40mm_HandSolder, F.Cu at (443.5, 4.32)
- added R20: 100k, Resistor_SMD:R_0805_2012Metric_Pad1.20x1.40mm_HandSolder, F.Cu at (443.8, -1.27)
- added R21: 200k, Resistor_SMD:R_0805_2012Metric_Pad1.20x1.40mm_HandSolder, F.Cu at (443.8, -3.30)
- added R22: 100k, Resistor_SMD:R_0805_2012Metric_Pad1.20x1.40mm_HandSolder, F.Cu at (239.1, 78.4)
- added R23: 100k, Resistor_SMD:R_0805_2012Metric_Pad1.20x1.40mm_HandSolder, F.Cu at (239.1, 81.4)
- added R24: 10k, Resistor_SMD:R_0805_2012Metric_Pad1.20x1.40mm_HandSolder, F.Cu at (201.2, 52.6)
- added R25: 10k, Resistor_SMD:R_0805_2012Metric_Pad1.20x1.40mm_HandSolder, F.Cu at (201.2, 55.5)
- added R26: 10k, Resistor_SMD:R_0805_2012Metric_Pad1.20x1.40mm_HandSolder, F.Cu at (201.2, 58.5)
- added R27: 113R, Resistor_SMD:R_0805_2012Metric_Pad1.20x1.40mm_HandSolder, F.Cu at (262.7, 36.1)
- added R28: 147R, Resistor_SMD:R_0805_2012Metric_Pad1.20x1.40mm_HandSolder, F.Cu at (262.7, 39.0)
- added R3: 10k, Resistor_SMD:R_0805_2012Metric_Pad1.20x1.40mm_HandSolder, F.Cu at (196.4, 55.5)
- added R4: 100k, Resistor_SMD:R_0805_2012Metric_Pad1.20x1.40mm_HandSolder, F.Cu at (196.4, 58.5)
- added R5: 100k, Resistor_SMD:R_0805_2012Metric_Pad1.20x1.40mm_HandSolder, F.Cu at (196.4, 61.4)
- added R6: 47k, Resistor_SMD:R_0805_2012Metric_Pad1.20x1.40mm_HandSolder, F.Cu at (196.4, 64.4)
- added R7: 10k, Resistor_SMD:R_0805_2012Metric_Pad1.20x1.40mm_HandSolder, F.Cu at (201.2, 49.6)
- added R8: 680R, Resistor_SMD:R_0603_1608Metric, F.Cu at (346.2, 15.3)
- added R9: 4k7, Resistor_SMD:R_0805_2012Metric_Pad1.20x1.40mm_HandSolder, F.Cu at (372.5, -1.98)
- added SW1: PEC09-2320F-S0015, Rotary_Encoder:RotaryEncoder_Bourns_Horizontal_PEC09-2xxxF-Sxxxx, F.Cu at (109.1, 77.5)
- added TP1: TestPoint_Small, TestPoint:TestPoint_Pad_D1.5mm, F.Cu at (348.9, 15.0)
- added TP10: TestPoint_Small, TestPoint:TestPoint_Pad_D1.5mm, F.Cu at (225.9, 53.5)
- added TP11: TestPoint_Small, TestPoint:TestPoint_Pad_D1.5mm, F.Cu at (225.9, 57.0)
- added TP12: TestPoint_Small, TestPoint:TestPoint_Pad_D1.5mm, F.Cu at (229.4, 49.9)
- added TP13: TestPoint_Small, TestPoint:TestPoint_Pad_D1.5mm, F.Cu at (252.8, 70.5)
- added TP14: TestPoint_Small, TestPoint:TestPoint_Pad_D1.5mm, F.Cu at (453.6, 8.38)
- added TP15: TestPoint_Small, TestPoint:TestPoint_Pad_D1.5mm, F.Cu at (453.6, -5.33)
- added TP16: TestPoint_Small, TestPoint:TestPoint_Pad_D1.5mm, F.Cu at (229.4, 53.5)
- added TP17: TestPoint_Small, TestPoint:TestPoint_Pad_D1.5mm, F.Cu at (229.4, 57.0)
- added TP18: TestPoint_Small, TestPoint:TestPoint_Pad_D1.5mm, F.Cu at (233.0, 49.9)
- added TP19: TestPoint_Small, TestPoint:TestPoint_Pad_D1.5mm, F.Cu at (233.0, 53.5)
- added TP2: TestPoint_Small, TestPoint:TestPoint_Pad_D1.5mm, F.Cu at (259.3, 52.4)
- added TP20: TestPoint_Small, TestPoint:TestPoint_Pad_D1.5mm, F.Cu at (233.0, 57.0)
- added TP3: TestPoint_Small, TestPoint:TestPoint_Pad_D1.5mm, F.Cu at (249.3, 66.9)
- added TP4: TestPoint_Small, TestPoint:TestPoint_Pad_D1.5mm, F.Cu at (249.3, 70.5)
- added TP5: TestPoint_Small, TestPoint:TestPoint_Pad_D1.5mm, F.Cu at (252.8, 66.9)
- added TP6: TestPoint_Small, TestPoint:TestPoint_Pad_D1.5mm, F.Cu at (222.3, 49.9)
- added TP7: TestPoint_Small, TestPoint:TestPoint_Pad_D1.5mm, F.Cu at (222.3, 53.5)
- added TP8: TestPoint_Small, TestPoint:TestPoint_Pad_D1.5mm, F.Cu at (222.3, 57.0)
- added TP9: TestPoint_Small, TestPoint:TestPoint_Pad_D1.5mm, F.Cu at (225.9, 49.9)
- added U1: IS25LP032D-JKLE, Package_SON:WSON-8-1EP_6x5mm_P1.27mm_EP3.4x4mm, F.Cu at (222.6, 43.0)
- added U2: XU316-1024-TQ128-C24, USB_to_I2S_Board:QFP40P1600X1600X120-129N, F.Cu at (360.2, 5.33)
- added U3: TPS62410DRCR, USB_to_I2S_Board:TPS62410DRCR, F.Cu at (444.0, 1.52)
- added U4: MAX809STRG, Package_TO_SOT_SMD:SOT-23, F.Cu at (250.0, 85.0)
- added U5: 74LVC2G07, Package_TO_SOT_SMD:SOT-363_SC-70-6, F.Cu at (238.7, 84.7)
- added Y1: FA-238 24MHz, Crystal:Crystal_SMD_3225-4Pin_3.2x2.5mm, F.Cu at (349.3, 18.0)
- J1: value Conn_01x30 -> UJ20-C-H-G-SMT-5-P16-TR; footprint Nathophone_Driverboard:CON_525593072_MOL -> USB_to_I2S_Board:SAMESKY_UJ20-C-H-G-SMT-5-P16-TR
- J2: value UJ20-C-H-G-SMT-5-P16-TR -> FTSH-110-01-F-DV-K; footprint USB_to_I2S_Board:SAMESKY_UJ20-C-H-G-SMT-5-P16-TR -> USB_to_I2S_Board:CON20_2X10_DUK_FTSH_SAI-M
- moved J2 248.3 mm to (211.0, 62.8)
- moved R1 219.7 mm to (196.4, 49.6)
- moved R2 219.7 mm to (196.4, 52.6)
- moved J1 168.8 mm to (105.1, 99.5), turned to -90 degrees
- moved CR1 161.0 mm to (111.3, 100.0), turned to 90 degrees
Connections:
- CR1 pad 1: /USB_D+ -> /Connectors_Misc/USB_D+
- CR1 pad 3: unconnected-(CR1-Pad3) -> /Connectors_Misc/USB_CC2
- CR1 pad 4: unconnected-(CR1-Pad4) -> /Connectors_Misc/USB_CC1
- CR1 pad 6: /USB_D- -> /Connectors_Misc/USB_D-
- R1 pad 1: Net-(J2-CC2) -> /Connectors_Misc/USB_CC2
- R2 pad 1: Net-(J2-CC1) -> /Connectors_Misc/USB_CC1
Routing:
- net /Connectors_Misc/USB_D+: track 0.00 -> 7.68 mm
- net /Connectors_Misc/USB_D-: track 0.00 -> 6.89 mm
- net GND: vias 0 -> 234
- added copper zone on In1.Cu, net GND
Other:
- copper layers 2 -> 4

Commit message: PLACED all footprints and GND zone
Parts:
- removed D1: LTST-C235KGKRKT, LED_SMD:LED_LiteOn_LTST-C235KGKRKT
- removed TP10, TP11, TP12, TP4, TP7, TP9: TestPoint_Small, TestPoint:TestPoint_Pad_D1.5mm
- added D2: XZMDKVG55W-8, USB_to_I2S_Board:LED_XZMDKVG55W-8, F.Cu at (123.4, 88.7)
- JP1: moved to B.Cu
- R27: value 113R -> 750R
- R28: value 147R -> 680R
- moved TP14 327.2 mm to (141.5, 106.7), turned to 90 degrees
- moved C15 326.3 mm to (145.6, 106.9)
- moved TP15 326.3 mm to (141.5, 89.6), turned to 180 degrees
- moved C16 322.7 mm to (145.6, 90.2)
- moved L1 319.0 mm to (145.8, 101.8), turned to -90 degrees
- moved L2 318.4 mm to (145.8, 95.2), turned to 90 degrees
- moved C14 317.6 mm to (141.2, 91.9)
- moved C17 317.6 mm to (137.5, 98.3)
- moved R18 317.6 mm to (141.1, 103.4)
- moved R19 317.6 mm to (141.1, 101.3)
- moved R20 317.6 mm to (141.3, 95.8)
- moved R21 317.6 mm to (141.3, 93.7)
- moved U3 317.6 mm to (141.6, 98.6)
- moved C13 240.0 mm to (154.7, 97.0), turned to 180 degrees
- moved R9 238.5 mm to (154.6, 94.9), turned to 0 degrees
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Connections:
- C37 pad 1: /Connectors_Misc/Rot_Enc_B -> Rot_Enc_B
- C38 pad 1: /Connectors_Misc/Rot_Enc_SW -> Rot_Enc_SW
- C39 pad 1: /Connectors_Misc/Rot_Enc_A -> Rot_Enc_A
- C4 pad 1: /Connectors_Misc/~{RST} -> ~{RST}
- CR1 pad 1: /Connectors_Misc/USB_D+ -> USB_D+
- CR1 pad 6: /Connectors_Misc/USB_D- -> USB_D-
- J1 pad A6: /Connectors_Misc/USB_D+ -> USB_D+
- J1 pad A7: /Connectors_Misc/USB_D- -> USB_D-
- J1 pad B6: /Connectors_Misc/USB_D+ -> USB_D+
- J1 pad B7: /Connectors_Misc/USB_D- -> USB_D-
- J2 pad 10: /Connectors_Misc/~{RST} -> ~{RST}
- J2 pad 12: /Connectors_Misc/XL_DN1 -> XL_DN1
- J2 pad 14: /Connectors_Misc/XL_DN0 -> XL_DN0
- J2 pad 16: /Connectors_Misc/XL_UP0 -> XL_UP0
- J2 pad 18: /Connectors_Misc/XL_UP1 -> XL_UP1
- J2 pad 2: /Connectors_Misc/TMS -> TMS
- J2 pad 4: /Connectors_Misc/TCK -> TCK
- J2 pad 6: /Connectors_Misc/TDO -> TDO
- J2 pad 8: /Connectors_Misc/TDI -> TDI
- J3 pad 13: /Connectors_Misc/SDATA -> SDATA
- J3 pad 17: /Connectors_Misc/SCLK -> SCLK
- J3 pad 19: /Connectors_Misc/LRCLK -> LRCLK
- J3 pad 21: /Connectors_Misc/MRCLK -> MRCLK
- J3 pad 5: /Connectors_Misc/GPIO -> GPIO
- J3 pad 6: /Connectors_Misc/~{SYS_RESET} -> ~{SYS_RESET}
- J4 pad 1: /Connectors_Misc/~{QSPI_CS} -> ~{QSPI_CS}
- J4 pad 10: /Connectors_Misc/MRCLK -> MRCLK
- J4 pad 2: /Connectors_Misc/~{SYS_RESET} -> ~{SYS_RESET}
- J4 pad 3: /Connectors_Misc/~{~{VBUS_DET}} -> ~{VBUS_DET}
- J4 pad 4: /Connectors_Misc/SDATA -> SDATA
- J4 pad 6: /Connectors_Misc/SCLK -> SCLK
- J4 pad 7: /Connectors_Misc/SDA -> SDA
- J4 pad 8: /Connectors_Misc/LRCLK -> LRCLK
- J4 pad 9: /Connectors_Misc/SCL -> SCL
- Q1 pad 3: /Connectors_Misc/~{~{VBUS_DET}} -> ~{VBUS_DET}
- R11 pad 2: /XMOS/SCL -> SCL
- R12 pad 1: /XMOS/XL_UP0 -> XL_UP0
- R13 pad 1: /XMOS/XL_UP1 -> XL_UP1
- R14 pad 1: /XMOS/SDATA -> SDATA
- R15 pad 1: /XMOS/LRCLK -> LRCLK
- R16 pad 1: /XMOS/SCLK -> SCLK
- R17 pad 1: /XMOS/MRCLK -> MRCLK
- R23 pad 1: /Power/~{SYS_RESET} -> ~{SYS_RESET}
- R24 pad 2: /Connectors_Misc/Rot_Enc_B -> Rot_Enc_B
- R25 pad 2: /Connectors_Misc/Rot_Enc_A -> Rot_Enc_A
- R26 pad 2: /Connectors_Misc/Rot_Enc_SW -> Rot_Enc_SW
- R3 pad 2: /Connectors_Misc/~{RST} -> ~{RST}
- R6 pad 2: /Connectors_Misc/~{~{VBUS_DET}} -> ~{VBUS_DET}
- R7 pad 2: /Connectors_Misc/~{QSPI_CS} -> ~{QSPI_CS}
- R9 pad 2: /XMOS/SDA -> SDA
- SW1 pad A: /Connectors_Misc/Rot_Enc_A -> Rot_Enc_A
- SW1 pad B: /Connectors_Misc/Rot_Enc_B -> Rot_Enc_B
- SW1 pad S1: /Connectors_Misc/Rot_Enc_SW -> Rot_Enc_SW
- TP13 pad 1: /Power/~{RST} -> ~{RST}
- TP16 pad 1: /Connectors_Misc/QSPI_CLK -> QSPI_CLK
- TP17 pad 1: /Connectors_Misc/QSPI_D0 -> QSPI_D0
- TP18 pad 1: /Connectors_Misc/QSPI_D1 -> QSPI_D1
- TP19 pad 1: /Connectors_Misc/QSPI_D2 -> QSPI_D2
- TP20 pad 1: /Connectors_Misc/QSPI_D3 -> QSPI_D3
- TP5 pad 1: /Power/~{SYS_RESET} -> ~{SYS_RESET}
- TP8 pad 1: /Connectors_Misc/~{~{VBUS_DET}} -> ~{VBUS_DET}
- U1 pad 1: /Connectors_Misc/~{QSPI_CS} -> ~{QSPI_CS}
- U1 pad 2: /Connectors_Misc/QSPI_D1 -> QSPI_D1
- U1 pad 3: /Connectors_Misc/QSPI_D2 -> QSPI_D2
- U1 pad 5: /Connectors_Misc/QSPI_D0 -> QSPI_D0
- U1 pad 6: /Connectors_Misc/QSPI_CLK -> QSPI_CLK
- U1 pad 7: /Connectors_Misc/QSPI_D3 -> QSPI_D3
- U2 pad 1: /XMOS/QSPI_D2 -> QSPI_D2
- U2 pad 127: /XMOS/QSPI_D0 -> QSPI_D0
- U2 pad 128: /XMOS/QSPI_D1 -> QSPI_D1
- U2 pad 2: /XMOS/~{QSPI_CS} -> ~{QSPI_CS}
- U2 pad 3: /XMOS/QSPI_D3 -> QSPI_D3
- U2 pad 36: /XMOS/TDI -> TDI
- U2 pad 37: /XMOS/TDO -> TDO
- U2 pad 4: /XMOS/QSPI_CLK -> QSPI_CLK
- U2 pad 44: /XMOS/TMS -> TMS
- U2 pad 51: /XMOS/TCK -> TCK
- U2 pad 59: /XMOS/USB_D- -> USB_D-
- U2 pad 60: /XMOS/USB_D+ -> USB_D+
- U2 pad 66: /XMOS/XL_DN1 -> XL_DN1
- U2 pad 67: /XMOS/XL_DN0 -> XL_DN0
- U2 pad 8: /XMOS/~{VBUS_DET} -> ~{VBUS_DET}
- U2 pad 81: /XMOS/GPIO -> GPIO
- U2 pad 82: /XMOS/Rot_Enc_A -> Rot_Enc_A
- U2 pad 83: /XMOS/Rot_Enc_B -> Rot_Enc_B
- U2 pad 84: /XMOS/Rot_Enc_SW -> Rot_Enc_SW
- U2 pad 93: /XMOS/SCL -> SCL
- U2 pad 94: /XMOS/SDA -> SDA
- U5 pad 1: /Power/~{RST} -> ~{RST}
- U5 pad 4: /Power/~{SYS_RESET} -> ~{SYS_RESET}
- U5 pad 6: /Power/~{SYS_RESET} -> ~{SYS_RESET}
Routing:
- net USB_D+: track 0.00 -> 7.68 mm
- net /Connectors_Misc/USB_D+: track 7.68 -> 0.00 mm
- net USB_D-: track 0.00 -> 6.89 mm
- net /Connectors_Misc/USB_D-: track 6.89 -> 0.00 mm
- net GND: vias 234 -> 221
- added copper zone on B.Cu, net GND
- added copper zone on F.Cu, net GND
- added copper zone on In2.Cu, net GND

Commit message: CONTINUED LAYOUT, MAIN Connections
Parts:
- moved R3 34.4 mm to (185.2, 94.0)
- moved C16 5.61 mm to (141.7, 94.2), turned to -90 degrees
- moved C15 5.41 mm to (141.7, 103.1), turned to 90 degrees
- moved TP15 4.40 mm to (145.8, 90.7), turned to 90 degrees
- moved TP14 4.28 mm to (145.8, 106.7), turned to 180 degrees
- moved R20 3.41 mm to (138.2, 94.5)
- moved R21 3.41 mm to (138.2, 92.5)
- moved C14 3.41 mm to (138.1, 90.7)
- moved R18 2.98 mm to (138.2, 104.1)
- moved R19 2.98 mm to (138.2, 102.1)
- moved TP13 2.40 mm to (184.2, 91.7)
- moved C17 1.55 mm to (136.0, 98.3)
- moved C4 1.02 mm to (150.1, 77.5), turned to 90 degrees
- moved TP5 0.51 mm to (188.5, 94.0)
- turned R28 to 180 degrees
Connections:
- U1 pad 9: (no net) -> GND
Routing:
- net +5V: track 0.00 -> 107.2 mm, vias 0 -> 11
- net USB_D-: track 6.89 -> 57.2 mm
- net USB_D+: track 7.68 -> 57.5 mm
- net GND: track 0.00 -> 27.2 mm, vias 221 -> 244
- net VDD: track 0.00 -> 22.1 mm
- net Rot_Enc_A: track 0.00 -> 18.7 mm
- net VBUS: track 0.00 -> 15.1 mm, vias 0 -> 2
- net +1V8: track 0.00 -> 14.9 mm
- net Rot_Enc_B: track 0.00 -> 14.4 mm
- net Net-(U2A-XOUT): track 0.00 -> 12.1 mm
- net Net-(U2A-XIN): track 0.00 -> 10.0 mm
- net +3.3V: track 0.00 -> 8.14 mm, vias 0 -> 2
- net Net-(U3-ADJ2): track 0.00 -> 8.13 mm
- net Rot_Enc_SW: track 0.00 -> 7.15 mm
- net Net-(U3-DEF_1): track 0.00 -> 6.11 mm
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- added copper zone on F.Cu, net +5V
- added copper zone on F.Cu, net Net-(U3-SW1)
- added copper zone on F.Cu, net Net-(U3-SW2)

Commit message: CONTINUED main layout
Parts:
- moved R6 51.7 mm to (180.3, 107.2)
- moved TP13 32.2 mm to (155.7, 76.7)
- moved TP8 5.57 mm to (136.4, 106.9)
Routing:
- net +3.3V: track 8.14 -> 201.2 mm, vias 2 -> 15
- net VDD: track 22.1 -> 190.0 mm, vias 0 -> 23
- net +1V8: track 14.9 -> 134.2 mm, vias 0 -> 12
- net /Power/~{3.3V_RESET}: track 0.00 -> 75.0 mm, vias 2 -> 4
- net ~{VBUS_DET}: track 5.04 -> 79.5 mm, vias 0 -> 3
- net ~{SYS_RESET}: track 0.00 -> 31.9 mm, vias 0 -> 2
- net MRCLK: track 0.00 -> 23.1 mm, vias 0 -> 2
- net SCLK: track 0.00 -> 17.9 mm, vias 0 -> 2
- net +5V: track 107.2 -> 124.0 mm, vias 11 -> 17
- net VBUS: track 15.1 -> 26.5 mm
- net /XMOS/MCLK_PIN: track 0.00 -> 9.32 mm, vias 0 -> 1
- net LRCLK: track 0.00 -> 8.63 mm, vias 0 -> 1
- net ~{QSPI_CS}: track 0.00 -> 7.09 mm
- net ~{RST}: track 3.07 -> 9.42 mm
- net /Connectors_Misc/USB_CC1: track 3.12 -> 8.66 mm
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
Commit message: COMPLETED first version of Layout
Parts:
- moved TP6 4.10 mm to (189.2, 79.5)
Routing:
- net ~{RST}: track 9.42 -> 62.4 mm, vias 0 -> 3
- net SCL: track 3.80 -> 49.5 mm, vias 0 -> 2
- net SDA: track 4.47 -> 47.7 mm, vias 0 -> 3
- net Rot_Enc_SW: track 7.15 -> 47.1 mm, vias 0 -> 2
- net GPIO: track 0.00 -> 39.0 mm
- net Rot_Enc_A: track 18.7 -> 53.5 mm, vias 0 -> 2
- net Rot_Enc_B: track 14.4 -> 46.0 mm, vias 0 -> 2
- net Net-(U2A-X1D53): track 0.00 -> 31.2 mm, vias 0 -> 2
- net Net-(U2A-X1D54): track 0.00 -> 31.1 mm, vias 0 -> 2
- net TDI: track 0.00 -> 27.9 mm, vias 0 -> 2
- net TDO: track 0.00 -> 27.8 mm, vias 0 -> 2
- net TMS: track 0.00 -> 27.2 mm, vias 0 -> 2
- net TCK: track 0.00 -> 24.1 mm, vias 0 -> 2
- net MRCLK: track 23.1 -> 47.0 mm, vias 2 -> 3
- net QSPI_D3: track 0.00 -> 23.0 mm, vias 0 -> 2
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Other:
- board text added: "+1.8V"
- board text added: "+3.3V"
- board text added: "+5V"
- board text added: "Nathophone USB to I2S Module V.1, 2026 by Nathanael Gubler"
- board text added: "VDD"
- board text added: "~{QSPI_CS} ~{SYS_RESET} VBUS_DET SDATA GND SCLK SDA LRCLK SCL MRCLK"
- board text added: "~{RST}"
- board text added: "~{SYS_RESET}"
- board text added: "~{VBUS_DET}"
