File: USBtoI2S_board/nathophone_USBtoI2S/nathophone_USBtoI2S.kicad_sch (KiCad schematic)
At the start: 0 parts

Commit message: ADDED USBtoI2S board design files
Other:
- company: (none) -> Private
- title: (none) -> Nathophone USB_to_I2S Module
Changed lines of the file:
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@@
 	(generator_version "10.0")
 	(paper "A4")
+	(title_block
+		(title "Nathophone USB_to_I2S Module")
+		(date "2026-08-08")
+		(rev "v3")
+		(company "Private")
+	)
 	(sheet
 		(at 29.21 28.575)
